Commit message: teacher's day

File: CrazySim/ros2_ws/src/test_pkg/models/model.urdf (robot description, URDF)
Before this commit: robot manipulator, 5 links, 4 joints
Links:
- link curvature_link: geometry visual mesh filename=pacasdfkage://test_pkg/models/meshes/curvature.dae scale=0.01 0.02 0.02
- link sphere_link: geometry visual mesh filename=packagasdfe://test_pkg/models/meshes/sphere.dae scale=0.006 0.006 0.006

Commit message: jungsanghwa

File: CrazySim/ros2_ws/src/test_pkg/models/model.urdf (robot description, URDF)
Before this commit: robot manipulator, 5 links, 4 joints
Links:
- link curvature_link: geometry visual mesh filename=package://test_pkg/models/meshes/curvature.dae scale=0.01 0.02 0.02
- link sphere_link: geometry visual mesh filename=package://test_pkg/models/meshes/sphere.dae scale=0.006 0.006 0.006
